File: crossover/X-over for bookshelf-1/X-over for bookshelf-1.kicad_pcb (KiCad board)
At the start: 2 copper layers, 121.9 x 121.9 mm, 10 parts, among them J1 Screw_Terminal_01x02, J2 Screw_Terminal_01x04

Commit message: adding holes
Parts:
- added REF**: MountingHole_3mm, MountingHole:MountingHole_3mm, F.Cu at (182.9, 121.9)
- added REF**: MountingHole_4.3mm_M4, MountingHole:MountingHole_4.3mm_M4, F.Cu at (152.4, 137.2)
- added REF**: MountingHole_4.3mm_M4, MountingHole:MountingHole_4.3mm_M4, F.Cu at (124.5, 27.9)
- added REF**: MountingHole_3mm, MountingHole:MountingHole_3mm, F.Cu at (144.8, 35.6)
- added REF**: MountingHole_3mm, MountingHole:MountingHole_3mm, F.Cu at (76.2, 27.9)
- added REF**: MountingHole_3mm, MountingHole:MountingHole_3mm, F.Cu at (167.6, 132.1)
- added REF**: MountingHole_3mm, MountingHole:MountingHole_3mm, F.Cu at (96.5, 48.3)
- added REF**: MountingHole_4.3mm_M4, MountingHole:MountingHole_4.3mm_M4, F.Cu at (73.7, 104.1)
- added REF**: MountingHole_3mm, MountingHole:MountingHole_3mm, F.Cu at (144.8, 55.9)
- J1: value Screw_Terminal_01x02 -> Conn_01x02_Pin; footprint Connector_Wire:SolderWire-0.5sqmm_1x02_P4.6mm_D0.9mm_OD2.1mm -> Connector_Wire:SolderWire-1sqmm_1x02_P7.8mm_D1.4mm_OD3.9mm
- J2: value Screw_Terminal_01x04 -> Conn_01x04_Pin; footprint Connector_Wire:SolderWire-0.5sqmm_1x04_P4.6mm_D0.9mm_OD2.1mm -> Connector_Wire:SolderWire-1sqmm_1x04_P7.8mm_D1.4mm_OD3.9mm
- moved J2 25.3 mm to (170.2, 107.0), turned to 90 degrees
- moved L1 9.41 mm to (175.3, 138.9)
- moved J1 7.83 mm to (148.5, 127.0), turned to 0 degrees
- moved L2 5.08 mm to (131.7, 45.7)
- moved C3 3.44 mm to (152.4, 120.1)
- moved C1 2.54 mm to (177.8, 74.4)
Connections:
- C1 pad 2: Net-(J1-Pin_1) -> Net-(J1-Pin_2)
- C2 pad 1: Net-(J2-Pin_1) -> Net-(J2-Pin_4)
- C3 pad 2: Net-(J2-Pin_1) -> Net-(J2-Pin_4)
- L1 pad 1: Net-(J1-Pin_1) -> Net-(J1-Pin_2)
- L1 pad 2: Net-(J2-Pin_4) -> Net-(J2-Pin_1)
- L2 pad 1: Net-(J1-Pin_2) -> Net-(J1-Pin_1)
- R2 pad 1: Net-(J1-Pin_2) -> Net-(J1-Pin_1)
Routing:
- net Net-(J1-Pin_1): track 138.9 -> 190.1 mm
- net Net-(J1-Pin_2): track 191.7 -> 149.9 mm
- net Net-(J2-Pin_1): track 51.4 -> 10.1 mm
- net Net-(J2-Pin_4): track 12.2 -> 51.1 mm
- net Net-(C2-Pad2): track 87.1 -> 79.6 mm
- net Net-(L3-Pad2): track 74.8 -> 79.0 mm
- net Net-(J2-Pin_2): track 106.6 -> 110.3 mm
- net Net-(C3-Pad1): track 24.3 -> 22.7 mm
Other:
- board text added: "PCM mounting hole"
- board text added: "T+"
- board text added: "T-"
- board text added: "V+"
- board text added: "V-"
- board text added: "W+"
- board text added: "W-"
